File: Kicad/2 connector Sensor Board/2 connector Sensor Board.kicad_pcb (KiCad board)
At the start: 2 copper layers, 10 x 20 mm, 11 parts, among them J1 SPI, J15 TE 3-2363962-0 Connector, J2 7 pin FPC 0.3mm Panasonic Y3b, J3 free pins, J4 TE 3-2363962-0 Connector, J5 7 pin FPC 0.3mm Panasonic Y3b, J7 JST SH

Commit message: Added LCSC part numbers, DNP attr, and exported Gerbers
Connections:
- net CS1 renamed CS5
- net CS2 renamed CS6
- net CS3 renamed CS7
- net CS4 renamed CS8
Changed lines of the file:
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@@
 		)
 		(pad_to_mask_clearance 0.05)
-		(solder_mask_min_width 0.1)
 		(allow_soldermask_bridges_in_footprints yes)
 		(pcbplotparams
@@
 	(net 3 "VDD")
 	(net 4 "MISO1")
-	(net 5 "CS1")
+	(net 5 "CS5")
 	(net 6 "SCK1")
-	(net 7 "CS2")
+	(net 7 "CS8")
 	(net 8 "Free1")
 	(net 9 "SCL1")
@@
 	(net 11 "RS485-")
 	(net 12 "SDA1")
-	(net 13 "CS3")
-	(net 14 "CS4")
+	(net 13 "CS7")
+	(net 14 "CS6")
 	(net 15 "Free2")
 	(footprint "Connector_PinHeader_1.27mm:PinHeader_1x05_P1.27mm_Vertical"
@@
 			)
 		)
+		(property "LCSC" "C160404"
+			(at 0 0 0)
+			(layer "F.SilkS")
+			(hide yes)
+			(effects
+				(font
+					(size 1.27 1.27)
+					(thickness 0.15)
+				)
+			)
+		)
 		(property ki_fp_filters "Connector*:*_1x??-1MP*")
 		(sheetname "Root")
@@
 		(tags "resistor")
 		(property "Reference" "R2"
-			(at 0 -1.17 270)
+			(at 0 -1.17 -90)
 			(layer "F.SilkS")
 			(hide yes)
@@
 			)
 		)
+		(property "LCSC" "C25744"
+			(at 0 0 0)
+			(layer "F.SilkS")
+			(hide yes)
+			(effects
+				(font
+					(size 1.27 1.27)
+					(thickness 0.15)
+				)
+			)
+		)
 		(property ki_fp_filters "R_*")
 		(sheetname "Root")
@@
 			(layers "F.Cu" "F.Paste" "F.Mask")
 			(roundrect_rratio 0.25)
-			(net 7 "CS2")
+			(net 14 "CS6")
 			(pintype "passive")
 		)
@@
 		(tags "Through hole pin header THT 1x04 1.27mm single row")
 		(property "Reference" "J3"
-			(at 0 -1.695 270)
+			(at 0 -1.695 -90)
 			(layer "F.SilkS")
 			(hide yes)
@@
 			(layers "*.Cu" "*.Mask")
 			(remove_unused_layers no)
-			(net 13 "CS3")
+			(net 13 "CS7")
 			(pinfunction "Pin_1")
 			(pintype "passive")
@@
 			(layers "*.Cu" "*.Mask")
 			(remove_unused_layers no)
-			(net 14 "CS4")
+			(net 7 "CS8")
 			(pinfunction "Pin_2")
 			(pintype "passive")
@@
 		(sheetname "Root")
 		(sheetfile "2 connector Sensor Board.kicad_sch")
-		(attr smd)
+		(attr smd dnp)
 		(fp_rect
 			(start 0.49 -1.64)
@@
 			(size 0.23 0.44)
 			(layers "F.Cu" "F.Mask")
-			(net 5 "CS1")
+			(net 5 "CS5")
 			(pinfunction "Pin_5")
 			(pintype "passive")
@@
 		(tags "resistor")
 		(property "Reference" "R4"
-			(at 0 -1.17 270)
+			(at 0 -1.17 -90)
 			(layer "F.SilkS")
 			(hide yes)
@@
 			)
 		)
+		(property "LCSC" "C25744"
+			(at 0 0 0)
+			(layer "F.SilkS")
+			(hide yes)
+			(effects
+				(font
+					(size 1.27 1.27)
+					(thickness 0.15)
+				)
+			)
+		)
 		(property ki_fp_filters "R_*")
 		(sheetname "Root")
@@
 			(layers "F.Cu" "F.Paste" "F.Mask")
 			(roundrect_rratio 0.25)
-			(net 5 "CS1")
+			(net 5 "CS5")
 			(pintype "passive")
 		)
@@
 		(sheetname "Root")
 		(sheetfile "2 connector Sensor Board.kicad_sch")
-		(attr smd)
+		(attr smd dnp)
 		(fp_rect
 			(start -1.01 1.07)
@@
 			(size 0.23 0.44)
 			(layers "F.Cu" "F.Mask")
-			(net 7 "CS2")
+			(net 14 "CS6")
 			(pinfunction "Pin_5")
 			(pintype "passive")
@@
 			)
 		)
+		(property "LCSC" "C425104"
+			(at 0 0 0)
+			(layer "B.SilkS")
+			(hide yes)
+			(effects
+				(font
+					(size 1.27 1.27)
+					(thickness 0.15)
+				)
+			)
+		)
 		(property ki_fp_filters "Connector*:*_2x??-1MP*")
 		(sheetname "Root")
@@
 			(size 0.23 0.65)
 			(layers "B.Cu" "B.Paste" "B.Mask")
-			(net 13 "CS3")
+			(net 13 "CS7")
 			(pinfunction "Pin_4")
 			(pintype "passive")
@@
 			(size 0.23 0.65)
 			(layers "B.Cu" "B.Paste" "B.Mask")
-			(net 14 "CS4")
+			(net 7 "CS8")
 			(pinfunction "Pin_6")
 			(pintype "passive")
@@
 			(size 0.23 0.65)
 			(layers "B.Cu" "B.Paste" "B.Mask")
-			(net 14 "CS4")
+			(net 7 "CS8")
 			(pinfunction "Pin_25")
 			(pintype "passive")
@@
 			(size 0.23 0.65)
 			(layers "B.Cu" "B.Paste" "B.Mask")
-			(net 13 "CS3")
+			(net 13 "CS7")
 			(pinfunction "Pin_27")
 			(pintype "passive")
@@
 			)
 		)
+		(property "LCSC" "C425104"
+			(at 0 0 0)
+			(layer "B.SilkS")
+			(hide yes)
+			(effects
+				(font
+					(size 1.27 1.27)
+					(thickness 0.15)
+				)
+			)
+		)
 		(property ki_fp_filters "Connector*:*_2x??-1MP*")
 		(sheetname "Root")
@@
 			(size 0.23 0.65)
 			(layers "B.Cu" "B.Paste" "B.Mask")
-			(net 5 "CS1")
+			(net 5 "CS5")
 			(pinfunction "Pin_4")
 			(pintype "passive")
@@
 			(size 0.23 0.65)
 			(layers "B.Cu" "B.Paste" "B.Mask")
-			(net 7 "CS2")
+			(net 14 "CS6")
 			(pinfunction "Pin_6")
 			(pintype "passive")
@@
 			(size 0.23 0.65)
 			(layers "B.Cu" "B.Paste" "B.Mask")
-			(net 7 "CS2")
+			(net 14 "CS6")
 			(pinfunction "Pin_25")
 			(pintype "passive")
@@
 			(size 0.23 0.65)
 			(layers "B.Cu" "B.Paste" "B.Mask")
-			(net 5 "CS1")
+			(net 5 "CS5")
 			(pinfunction "Pin_27")
 			(pintype "passive")
@@
 	)
 	(segment
-		(start 141.3 103.7)
-		(end 140.75 104.25)
-		(width 0.16)
-		(layer "F.Cu")
-		(net 7)
-	)
-	(segment
-		(start 140.75 108.05)
-		(end 140.75 104.25)
-		(width 0.16)
-		(layer "F.Cu")
-		(net 7)
-	)
-	(segment
-		(start 142.955002 110.255002)
-		(end 140.75 108.05)
-		(width 0.16)
-		(layer "F.Cu")
-		(net 7)
-	)
-	(segment
-		(start 140.3 101.71)
-		(end 141.3 102.71)
-		(width 0.16)
-		(layer "F.Cu")
-		(net 7)
-	)
-	(segment
-		(start 140.75 104.25)
-		(end 140.06 104.25)
+		(start 144.83 97.8)
+		(end 144.09 98.54)
 		(width 0.16)
-		(layer "F.Cu")
+		(layer "B.Cu")
 		(net 7)
 	)
 	(segment
-		(start 145.66 110.255002)
-		(end 142.955002 110.255002)
+		(start 141.983481 98.54)
+		(end 141.5 98.056519)
 		(width 0.16)
-		(layer "F.Cu")
+		(layer "B.Cu")
 		(net 7)
 	)
 	(segment
-		(start 146.2 109.715002)
-		(end 145.66 110.255002)
+		(start 141.5 98.056519)
+		(end 141.5 97.180832)
 		(width 0.16)
-		(layer "F.Cu")
+		(layer "B.Cu")
 		(net 7)
 	)
 	(segment
-		(start 141.3 102.71)
-		(end 141.3 103.7)
+		(start 142.51 96.170832)
+		(end 142.51 95.68)
 		(width 0.16)
-		(layer "F.Cu")
-		(net 7)
-	)
-	(via
-		(at 146.2 109.715002)
-		(size 0.6)
-		(drill 0.3)
-		(layers "F.Cu" "B.Cu")
+		(layer "B.Cu")
 		(net 7)
 	)
 	(segment
-		(start 146.51 108.93)
-		(end 146.51 109.405002)
+		(start 144.09 98.54)
+		(end 141.983481 98.54)
 		(width 0.16)
 		(layer "B.Cu")
@@
 	)
 	(segment
-		(start 146.51 109.405002)
-		(end 146.2 109.715002)
+		(start 141.5 97.180832)
+		(end 142.51 96.170832)
 		(width 0.16)
 		(layer "B.Cu")
@@
 	)
 	(segment
-		(start 144.83 97.8)
-		(end 144.09 98.54)
+		(start 141.3 103.7)
+		(end 140.75 104.25)
 		(width 0.16)
-		(layer "B.Cu")
+		(layer "F.Cu")
 		(net 14)
 	)
 	(segment
-		(start 141.983481 98.54)
-		(end 141.5 98.056519)
+		(start 140.75 108.05)
+		(end 140.75 104.25)
 		(width 0.16)
-		(layer "B.Cu")
+		(layer "F.Cu")
 		(net 14)
 	)
 	(segment
-		(start 141.5 98.056519)
-		(end 141.5 97.180832)
+		(start 142.955002 110.255002)
+		(end 140.75 108.05)
 		(width 0.16)
-		(layer "B.Cu")
+		(layer "F.Cu")
 		(net 14)
 	)
 	(segment
-		(start 142.51 96.170832)
-		(end 142.51 95.68)
+		(start 140.3 101.71)
+		(end 141.3 102.71)
 		(width 0.16)
-		(layer "B.Cu")
+		(layer "F.Cu")
 		(net 14)
 	)
 	(segment
-		(start 144.09 98.54)
-		(end 141.983481 98.54)
+		(start 140.75 104.25)
+		(end 140.06 104.25)
+		(width 0.16)
+		(layer "F.Cu")
+		(net 14)
+	)
+	(segment
+		(start 145.66 110.255002)
+		(end 142.955002 110.255002)
+		(width 0.16)
+		(layer "F.Cu")
+		(net 14)
+	)
+	(segment
+		(start 146.2 109.715002)
+		(end 145.66 110.255002)
+		(width 0.16)
+		(layer "F.Cu")
+		(net 14)
+	)
+	(segment
+		(start 141.3 102.71)
+		(end 141.3 103.7)
+		(width 0.16)
+		(layer "F.Cu")
+		(net 14)
+	)
+	(via
+		(at 146.2 109.715002)
+		(size 0.6)
+		(drill 0.3)
+		(layers "F.Cu" "B.Cu")
+		(net 14)
+	)
+	(segment
+		(start 146.51 108.93)
+		(end 146.51 109.405002)
 		(width 0.16)
 		(layer "B.Cu")
@@
 	)
 	(segment
-		(start 141.5 97.180832)
-		(end 142.51 96.170832)
+		(start 146.51 109.405002)
+		(end 146.2 109.715002)
 		(width 0.16)
 		(layer "B.Cu")
