File: Kicad/Verticale Sensor Spacer/Verticale Sensor Spacer.kicad_sch (KiCad schematic)
At the start: 2 parts, among them J1 TE 3-2363961-0 Connector, J15 TE 3-2363962-0 Connector

Commit message: Added LCSC part numbers, DNP attr, and exported Gerbers
Parts:
- J1: LCSC (none) -> C425103
- J15: LCSC (none) -> C425104
Changed lines of the file:
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@@
+			)
+		)
+		(property "LCSC" "C425104"
+			(at 119.126 82.042 0)
+			(effects
+				(font
+					(size 1.27 1.27)
+				)
+				(hide yes)
 			)
 		)
@@
 			(effects
 				(font
+					(size 1.27 1.27)
+				)
+				(hide yes)
+			)
+		)
+		(property "LCSC" "C425103"
+			(at 186.436 82.042 0)
+			(effects
+				(font
