File: Hardware/Drivers/DRV8213 brushed Motor Driver/DRV8213 brushed Motor Driver.kicad_sch (KiCad schematic)
At the start: 26 parts, among them J1 Keystone 3569, J10 1.27mm pin header, J11 1.27mm pin header, J2 Keystone 3579, J3 Keystone 3579, J4 Keystone 3569, J5 Keystone 3569, J6 Keystone 3579, J7 Keystone 3579, J8 Keystone 3569, J9 JST PH 2mm horizontal, U1 DRV8213RTER, U2 LP2981-3.3

Commit message: Updated files for JLC DFM checks
Parts:
- J10, J11: now not fitted
- J9: LCSC C295747 -> C160237; Rotation Offset (none) -> 180
Changed lines of the file:
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@@
 		(in_bom yes)
 		(on_board yes)
-		(dnp no)
+		(dnp yes)
 		(property "Reference" "J10"
 			(at 76.2 73.6601 0)
@@
 			)
 		)
-		(property "LCSC" "C295747"
+		(property "LCSC" "C160237"
 			(at 147.32 59.6899 0)
+			(effects
+				(font
+					(size 1.27 1.27)
+				)
+				(hide yes)
+			)
+		)
+		(property "Rotation Offset" "180"
+			(at 146.05 59.69 0)
 			(effects
 				(font
@@
 		(in_bom yes)
 		(on_board yes)
-		(dnp no)
+		(dnp yes)
 		(property "Reference" "J11"
 			(at 37.592 119.888 0)
