File: Hardware/PSUs/2s 40A PSU and charger/2s 40A PSU and charger.kicad_sch (KiCad schematic)
At the start: 5 parts

Commit message: Added schematic PDFs for all boards
Other:
- company: (none) -> Author: Asher Edwards
Changed lines of the file:
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@@
 		(date "2024-12-23")
 		(rev "V1")
-		(comment 1 "Author: Asher Edwards")
+		(company "Author: Asher Edwards")
+		(comment 1 "Licensed under CERN-OHL-S")
 	)
 	(junction
