File: Hardware/PSUs/2s 40A PSU and charger/Battery Balancer.kicad_sch (KiCad schematic)
At the start: 22 parts, among them Q6 Vishay sir404dp, or SiR500DP, U1 BQ76905RGRR

Commit message: Updated files for JLC DFM checks
Parts:
- Q6: Rotation Offset (none) -> 270
Changed lines of the file:
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@@
+			)
+		)
+		(property "Rotation Offset" "270"
+			(at 77.47 110.49 90)
+			(effects
+				(font
+					(size 1.27 1.27)
+				)
+				(hide yes)
 			)
 		)

Commit message: Added schematic PDFs for all boards
Other:
- company: (none) -> Author: Asher Edwards
Changed lines of the file:
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@@
 		(date "2024-12-23")
 		(rev "V1")
-		(comment 1 "Author: Asher Edwards")
+		(company "Author: Asher Edwards")
+		(comment 1 "Licensed under CERN-OHL-S")
 	)
 	(junction
