File: Hardware/PSUs/2s 40A PSU and charger/Battery Charger.kicad_sch (KiCad schematic)
At the start: 40 parts

Commit message: Updated files for JLC DFM checks
Parts:
- L?: Rotation Offset (none) -> 90
- Q? (x4): Rotation Offset (none) -> 180
- Q?: LCSC (none) -> C3289487; Rotation Offset (none) -> 270
- U?: Rotation Offset (none) -> 270
Changed lines of the file:
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@@
 			)
 		)
+		(property "Rotation Offset" "180"
+			(at 173.99 113.03 0)
+			(effects
+				(font
+					(size 1.27 1.27)
+				)
+				(hide yes)
+			)
+		)
 		(pin "3"
 		)
@@
 			)
 		)
+		(property "Rotation Offset" "270"
+			(at 198.12 85.09 0)
+			(effects
+				(font
+					(size 1.27 1.27)
+				)
+				(hide yes)
+			)
+		)
+		(property "LCSC" "C3289487"
+			(at 198.12 85.09 0)
+			(effects
+				(font
+					(size 1.27 1.27)
+				)
+				(hide yes)
+			)
+		)
 		(pin "1"
 		)
@@
 			)
 		)
+		(property "Rotation Offset" "180"
+			(at 173.99 95.25 0)
+			(effects
+				(font
+					(size 1.27 1.27)
+				)
+				(hide yes)
+			)
+		)
 		(pin "3"
 		)
@@
 			)
 		)
+		(property "Rotation Offset" "180"
+			(at 100.33 57.15 90)
+			(effects
+				(font
+					(size 1.27 1.27)
+				)
+				(hide yes)
+			)
+		)
 		(pin "3"
 		)
@@
 			)
 		)
+		(property "Rotation Offset" "90"
+			(at 187.96 107.95 90)
+			(effects
+				(font
+					(size 1.27 1.27)
+				)
+				(hide yes)
+			)
+		)
 		(pin "2"
 		)
@@
 			)
 		)
+		(property "Rotation Offset" "180"
+			(at 82.55 57.15 90)
+			(effects
+				(font
+					(size 1.27 1.27)
+				)
+				(hide yes)
+			)
+		)
 		(pin "3"
 		)
@@
 			(at 132.08 118.11 0)
 			(effects
+				(font
+					(size 1.27 1.27)
+				)
+				(hide yes)
+			)
+		)
+		(property "Rotation Offset" "270"
+			(at 132.08 118.11 0)
+			(effects

Commit message: Added schematic PDFs for all boards
Other:
- company: (none) -> Author: Asher Edwards
Changed lines of the file:
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@@
 		(date "2024-12-23")
 		(rev "V1")
-		(comment 1 "Author: Asher Edwards")
+		(company "Author: Asher Edwards")
+		(comment 1 "Licensed under CERN-OHL-S")
 	)
 	(junction
