File: Hardware/PSUs/2s 40A PSU and charger/Connectors.kicad_sch (KiCad schematic)
At the start: 18 parts, among them J1 Keystone 3579, J10 G-Switch-GT-USB-7025, J11 1.27mm 4 pin socket, J2 JST XH-S Balance Plug, J3 Keystone 3579, J4 Keystone 3569, J5 Keystone 3569, J6 Keystone 3579, J7 Keystone 3579, J8 Keystone 3569, J9 Keystone 3569

Commit message: Updated files for JLC DFM checks
Parts:
- D11: Position Offset (none) -> 0,0.4
- J10: Position Offset (none) -> 0,1.55
- J2: now not fitted
Changed lines of the file:
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@@
 		(in_bom yes)
 		(on_board yes)
-		(dnp no)
+		(dnp yes)
 		(property "Reference" "J2"
 			(at 74.93 157.48 0)
@@
 			)
 		)
+		(property "Position Offset" "0,0.4"
+			(at 76.2 69.85 0)
+			(effects
+				(font
+					(size 1.27 1.27)
+				)
+				(hide yes)
+			)
+		)
 		(pin "7"
 		)
@@
 			(effects
 				(font
+					(size 1.27 1.27)
+				)
+				(hide yes)
+			)
+		)
+		(property "Position Offset" "0,1.55"
+			(at 52.07 67.31 0)
+			(effects
+				(font

Commit message: Added schematic PDFs for all boards
Other:
- company: (none) -> Author: Asher Edwards
Changed lines of the file:
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@@
 		(date "2024-12-23")
 		(rev "V1")
-		(comment 1 "Author: Asher Edwards")
+		(company "Author: Asher Edwards")
+		(comment 1 "Licensed under CERN-OHL-S")
 	)
 	(junction
