File: Hardware/PSUs/2s 40A PSU and charger/MCU.kicad_sch (KiCad schematic)
At the start: 18 parts, among them J12 USB, U5 THVD1420DRLR, U6 CH32X035G8U6

Commit message: Updated files for JLC DFM checks
Parts:
- U6: Rotation Offset (none) -> 180
Changed lines of the file:
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@@
+			)
+		)
+		(property "Rotation Offset" "180"
+			(at 140.97 91.44 0)
+			(effects
+				(font
+					(size 1.27 1.27)
+				)
+				(hide yes)
 			)
 		)

Commit message: Added schematic PDFs for all boards
Other:
- company: ME -> Author: Asher Edwards
Changed lines of the file:
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@@
 		(date "2024-12-23")
 		(rev "V1")
-		(company "ME")
-		(comment 1 "Author: Asher Edwards")
+		(company "Author: Asher Edwards")
+		(comment 1 "Licensed under CERN-OHL-S")
 	)
 	(junction
